Commit message: Velodyne stuff

File: p4_ws/src/swarm_simulation/launch/kobuki.xacro (robot description, xacro)
@@ -10,4 +10,5 @@
   <!--<xacro:include filename="$(find turtlebot_description)/urdf/stacks/hexagons.urdf.xacro"/>-->
   <xacro:include filename="$(find swarm_simulation)/urdf/velodyne_hexagon.urdf.xacro"/>
+ <!--<xacro:include filename="$(find swarm_simulation)/urdf/velodyne.urdf.xacro"/>-->
   <!--<xacro:include filename="$(find turtlebot_description)/urdf/sensors/kinect.urdf.xacro"/>-->
   <!-- <xacro:include filename="$(find swarm_simulation)../../../velodyne_plugin/models/velodyne_hdl32/model.urdf.xacro"/> -->

File: p4_ws/src/swarm_simulation/urdf/velodyne_hexagon.urdf.xacro (robot description, xacro)
@@ -3,6 +3,8 @@
   Hexagon stacks
  -->
-<robot name="stack_hexagons" xmlns:xacro="http://ros.org/wiki/xacro">
+<robot name="stack_hexagons"
+  xmlns:xacro="http://ros.org/wiki/xacro">
   <xacro:include filename="$(find turtlebot_description)/urdf/common_properties.urdf.xacro"/>
+  <xacro:include filename="$(find swarm_simulation)/urdf/velodyne_hexagon.gazebo"/>
   <!-- Xacro properties -->
   <xacro:property name="M_SCALE" value="0.001"/>
@@ -31,7 +33,5 @@
         <mass value="0.008"/>
         <origin xyz="0 0 0" rpy="0 0 0"/>
-        <inertia ixx="0.000001686" ixy="0.0" ixz="0.0"
-                 iyy="0.000001686" iyz="0.0"
-                 izz="0.000000144"/>
+        <inertia ixx="0.000001686" ixy="0.0" ixz="0.0" iyy="0.000001686" iyz="0.0" izz="0.000000144"/>
       </inertial>
     </link>
@@ -59,7 +59,5 @@
         <mass value="0.012"/>
         <origin xyz="0 0 0"/>
-        <inertia ixx="0.000003805" ixy="0.0" ixz="0.0"
-                 iyy="0.000003805" iyz="0.0"
-                 izz="0.000000216"/>
+        <inertia ixx="0.000003805" ixy="0.0" ixz="0.0" iyy="0.000003805" iyz="0.0" izz="0.000000216"/>
       </inertial>
     </link>
@@ -87,7 +85,5 @@
         <mass value="0.060"/>
         <origin xyz="0 0 0"/>
-        <inertia ixx="0.000206991" ixy="0.0" ixz="0.0"
-                 iyy="0.000206991" iyz="0.0"
-                 izz="0.000001080"/>
+        <inertia ixx="0.000206991" ixy="0.0" ixz="0.0" iyy="0.000206991" iyz="0.0" izz="0.000001080"/>
       </inertial>
     </link>
@@ -115,7 +111,5 @@
         <mass value="0.020"/>
         <origin xyz="0 0 0"/>
-        <inertia ixx="0.000014782" ixy="0.0" ixz="0.0"
-                 iyy="0.000014782" iyz="0.0"
-                 izz="0.000000360"/>
+        <inertia ixx="0.000014782" ixy="0.0" ixz="0.0" iyy="0.000014782" iyz="0.0" izz="0.000000360"/>
       </inertial>
     </link>
@@ -126,4 +120,35 @@
     other, but there is no necessary reason to do so.
   -->
+    <xacro:macro name="velodyne" params="parent">
+    <joint name="velodyne_joint" type="fixed">
+      <origin xyz="0 0 0.4" rpy="0 0 0"/>
+      <parent link="${parent}"/>
+      <child link="velodyne_link"/>
+    </joint>
+    <link name="velodyne_link">
+      <visual>
+        <origin xyz="0 0 0" rpy="0 0 1.57"/>
+        <geometry>
+          <mesh filename="package://swarm_simulation/../meshes/velodyne_top.dae"/>
+        </geometry>
+      </visual>
+      <collision>
+        <origin xyz="0 0 0" rpy="0 0 0"/>
+        <geometry>
+          <cylinder length="0.006" radius="0.170"/>
+        </geometry>
+      </collision>
+      <inertial>
+        <mass value="0.520"/>
+        <origin xyz="0 0 0"/>
+        <inertia ixx="0.003328" ixy="0.0" ixz="0.0" iyy="0.003328" iyz="0.0" izz="0.006656" />
+      </inertial>
+    </link>
+    <gazebo>
+      <plugin name="velodyne_control" filename="libvelodyne_plugin.so">
+        <velocity>8</velocity>
+      </plugin>
+    </gazebo>
+  </xacro:macro>
   <xacro:macro name="stack_hexagons" params="parent">
     <stack_bottom_pole parent="${parent}" number="0" x_loc= "0.120" y_loc= "0.082" z_loc="0.1028"/>
@@ -133,4 +158,5 @@
     <stack_bottom_pole parent="${parent}" number="4" x_loc= "0.055" y_loc="-0.120" z_loc="0.1028"/>
     <stack_bottom_pole parent="${parent}" number="5" x_loc="-0.055" y_loc="-0.120" z_loc="0.1028"/>
+    <velodyne parent="${parent}"/>
     <joint name="plate_bottom_joint" type="fixed">
       <origin xyz="0.02364 0.0 0.1306" rpy="0 0 0"/>
@@ -154,7 +180,5 @@
         <mass value="0.520" />
         <origin xyz="0 0 0" />
-        <inertia ixx="0.003328" ixy="0.0" ixz="0.0"
-                 iyy="0.003328" iyz="0.0"
-                 izz="0.006656" />
+        <inertia ixx="0.003328" ixy="0.0" ixz="0.0" iyy="0.003328" iyz="0.0" izz="0.006656" />
       </inertial>
     </link>
@@ -184,7 +208,5 @@
         <mass value="0.520" />
         <origin xyz="0 0 0" />
-        <inertia ixx="0.003328" ixy="0.0" ixz="0.0"
-                 iyy="0.003328" iyz="0.0"
-                 izz="0.006656" />
+        <inertia ixx="0.003328" ixy="0.0" ixz="0.0" iyy="0.003328" iyz="0.0" izz="0.006656" />
       </inertial>
     </link>
@@ -193,6 +215,4 @@
     <stack_top_pole parent="${parent}" number="2" x_loc="-0.0381" y_loc= "0.1505" z_loc="0.2920"/>
     <stack_top_pole parent="${parent}" number="3" x_loc="-0.0381" y_loc="-0.1505" z_loc="0.2920"/>
-    <stack_3d_sensor_pole parent="${parent}" number="0" x_loc="-0.1024" y_loc= "0.098" z_loc="0.2372"/>
-    <stack_3d_sensor_pole parent="${parent}" number="1" x_loc="-0.1024" y_loc="-0.098" z_loc="0.2372"/>
     <joint name="plate_top_joint" type="fixed">
       <origin xyz="-0.01364 0.0  0.3966" rpy="0 0 0"/>
@@ -216,9 +236,8 @@
         <mass value="0.520"/>
         <origin xyz="0 0 0"/>
-        <inertia ixx="0.003328" ixy="0.0" ixz="0.0"
-                 iyy="0.003328" iyz="0.0"
-                 izz="0.006656" />
-      </inertial>
-    </link>
+        <inertia ixx="0.003328" ixy="0.0" ixz="0.0" iyy="0.003328" iyz="0.0" izz="0.006656" />
+      </inertial>
+    </link>
+    <!--
     <joint name="plate_top_velodyne_base" type="fixed">
       <origin xyz="-0.01364 0.0  0.3966" rpy="0 0 0"/>
@@ -242,11 +261,9 @@
         <mass value="0.520"/>
         <origin xyz="0 0 0"/>
-        <inertia ixx="0.003328" ixy="0.0" ixz="0.0"
-                 iyy="0.003328" iyz="0.0"
-                 izz="0.006656" />
+        <inertia ixx="0.003328" ixy="0.0" ixz="0.0" iyy="0.003328" iyz="0.0" izz="0.006656" />
       </inertial>
     </link>
     <joint name="plate_top_velodyne_top" type="fixed">
-      <origin xyz="0 0.0  0.05867" rpy="0 0 0"/>
+      <origin xyz="0 0.0  0.07867" rpy="0 0 0"/>
       <parent link="plate_top_velodyne_base"/>
       <child link="plate_top_velodyne_top"/>
@@ -254,5 +271,5 @@
     <link name="plate_top_velodyne_top">
       <visual>
-        <origin xyz="0 0 0" rpy="0 0 0"/>
+        <origin xyz="0 0 -0.02" rpy="0 0 1.57"/>
         <geometry>
           <mesh filename="package://swarm_simulation/../meshes/velodyne_top.dae"/>
@@ -260,17 +277,16 @@
       </visual>
       <collision>
-        <origin xyz="0.01364 0 0" rpy="0 0 0"/>
-        <geometry>
-          <cylinder length="0.006" radius="0.170"/>
-        </geometry>
-      </collision>
-      <inertial>
-        <mass value="0.520"/>
-        <origin xyz="0 0 0"/>
-        <inertia ixx="0.003328" ixy="0.0" ixz="0.0"
-                 iyy="0.003328" iyz="0.0"
-                 izz="0.006656" />
-      </inertial>
-    </link>
+        <origin xyz="0.01364 0 -0.02" rpy="0 0 1.57"/>
+        <geometry>
+          <cylinder length="0.006" radius="0.170"/>
+        </geometry>
+      </collision>
+      <inertial>
+        <mass value="0.520"/>
+        <origin xyz="0 0 0"/>
+        <inertia ixx="0.003328" ixy="0.0" ixz="0.0" iyy="0.003328" iyz="0.0" izz="0.006656" />
+      </inertial>
+    </link>
+    -->
   </xacro:macro>
 </robot>
